Commit message: open_manipulator.gazebo.xacro update open_manipulator.urdf.xacro update

File: open_manipulator_description/urdf/open_manipulator.gazebo.xacro (robot description, xacro)
@@ -50,5 +50,5 @@
     </plugin>
   </gazebo>
-  <!-- camera -->
+  <!-- camera
   <gazebo reference="camera_link">
     <sensor type="camera" name="intel_realsense_r200">
@@ -67,7 +67,7 @@
         <noise>
           <type>gaussian</type>
-          <!-- Noise is sampled independently per pixel on each frame.
+           Noise is sampled independently per pixel on each frame.
                That pixel's noise value is added to each of its color
-               channels, which at that point lie in the range [0,1]. -->
+               channels, which at that point lie in the range [0,1]. -.->
           <mean>0.0</mean>
           <stddev>0.007</stddev>
@@ -90,3 +90,45 @@
     </sensor>
   </gazebo>
+  -->
+  <!-- Camera -->
+  <gazebo reference="camera_link">
+    <sensor type="camera" name="camera1">
+      <update_rate>30.0</update_rate>
+      <visualize>false</visualize>
+      <camera name="head">
+        <horizontal_fov>1.3962634</horizontal_fov>
+        <image>
+          <width>640</width>
+          <height>480</height>
+          <format>R8G8B8</format>
+        </image>
+        <clip>
+          <near>0.1</near>
+          <far>25.0</far>
+        </clip>
+        <noise>
+          <type>gaussian</type>
+          <!-- Noise is sampled independently per pixel on each frame.
+               That pixel's noise value is added to each of its color
+               channels, which at that point lie in the range [0,1]. -->
+          <mean>0.0</mean>
+          <stddev>0.007</stddev>
+        </noise>
+      </camera>
+      <plugin name="camera_controller" filename="libgazebo_ros_camera.so">
+        <alwaysOn>true</alwaysOn>
+        <updateRate>0.0</updateRate>
+        <cameraName>head_camera</cameraName>
+        <imageTopicName>image_raw</imageTopicName>
+        <cameraInfoTopicName>camera_info</cameraInfoTopicName>
+        <frameName>camera_link_optical</frameName>
+        <hackBaseline>0.07</hackBaseline>
+        <distortionK1>0.0</distortionK1>
+        <distortionK2>0.0</distortionK2>
+        <distortionK3>0.0</distortionK3>
+        <distortionT1>0.0</distortionT1>
+        <distortionT2>0.0</distortionT2>
+      </plugin>
+    </sensor>
+  </gazebo>
 </robot>

File: open_manipulator_description/urdf/open_manipulator.urdf.xacro (robot description, xacro)
@@ -235,11 +235,44 @@
     </inertial>
   </link>
-  <!-- Realsense Camera Joint Position -->
-<!--   <joint name="camera_joint" type="fixed">
+  <!-- Camera -->
+  <joint type="fixed" name="camera_joint">
+    <origin xyz="0.1 0 0.1" rpy="0 0 0"/>
+    <child link="camera_link"/>
+    <parent link="end_effector_link"/>
     <axis xyz="0 1 0" />
-    <origin xyz="0.070 0.032 0.052" rpy="0 0 0"/>
-    <parent link="link5"/>
-    <child link="camera_link"/>
-  </joint>
-  <link name="camera_link"/> -->
+  </joint>
+  <link name='camera_link'>
+    <pose>0 0 0 0 0 0</pose>
+    <inertial>
+      <mass value="0.1"/>
+      <origin xyz="0 0 0" rpy="0 0 0"/>
+      <inertia
+          ixx="1e-6" ixy="0" ixz="0"
+          iyy="1e-6" iyz="0"
+          izz="1e-6"
+      />
+    </inertial>
+    <collision name='collision'>
+      <origin xyz="0 0 0" rpy="0 0 0"/>
+      <geometry>
+        <box size=".05 .05 .05"/>
+      </geometry>
+    </collision>
+    <visual name='camera_link_visual'>
+      <origin xyz="0 0 0" rpy="0 0 0"/>
+      <geometry>
+        <box size=".05 .05 .05"/>
+      </geometry>
+    </visual>
+  </link>
+  <gazebo reference="camera_link">
+    <material>Gazebo/Red</material>
+  </gazebo>
+  <joint type="fixed" name="camera_optical_joint">
+    <origin xyz="0 0 0" rpy="-1.5707 0 -1.5707"/>
+    <child link="camera_link_optical"/>
+    <parent link="camera_link"/>
+  </joint>
+  <link name="camera_link_optical">
+  </link>
 </robot>

Commit message: kamera+tartó modellje javítva, kamera jó helyen és jó irányba áll

File: open_manipulator_description/urdf/open_manipulator.gazebo.xacro (robot description, xacro)
@@ -95,5 +95,5 @@
     <sensor type="camera" name="camera1">
       <update_rate>30.0</update_rate>
-      <visualize>false</visualize>
+      <visualize>true</visualize>
       <camera name="head">
         <horizontal_fov>1.3962634</horizontal_fov>

File: open_manipulator_description/urdf/open_manipulator.urdf.xacro (robot description, xacro)
@@ -235,7 +235,7 @@
     </inertial>
   </link>
-  <!-- camera stand joint -->
+  <!-- camera joint -->
   <joint name="camera_joint" type="fixed">
-    <origin xyz="-0.0595 0 0.0380" rpy="${pi*0.5} ${pi*0.5} ${pi*1.5}"/>
+    <origin xyz="-0.0595 0 0.0510" rpy="0 0 0"/>
     <!--origin xyz="-0.0595 0 0.0430" rpy="${pi*0.5} 0 ${pi*1.5}"ez legyen, ha már jo a csavarkotes cad-je-->
     <parent link="end_effector_link"/>
@@ -245,12 +245,12 @@
   <link name="camera_link">
     <visual>
-      <origin xyz="0 0 0" rpy="0 0 0"/>
-      <geometry>
-        <mesh filename="package://open_manipulator_description/meshes/tartos_kamera.dae" scale="1 1 1"/>
+      <origin xyz="0 0 0.0150" rpy="0 0 ${pi*1}"/>
+      <geometry>
+        <mesh filename="package://open_manipulator_description/meshes/tartos_kamera3.dae" scale="1 1 1"/>
       </geometry>
       <material name="red"/>
      </visual>
     <inertial>
-      <origin xyz="0 0 0" />
+      <origin xyz="0 0 0.0150" rpy="0 0 ${pi*1}"/>
       <mass value="1.0e-03" />
       <inertia ixx="1.0e-03" ixy="0.0" ixz="0.0"
@@ -259,7 +259,7 @@
     </inertial>
     <collision name='collision'>
-      <origin xyz="0 0 0" rpy="0 0 0"/>
-      <geometry>
-        <mesh filename="package://open_manipulator_description/meshes/tartos_kamera.dae" scale="1 1 1"/>
+      <origin xyz="0 0 0.0150" rpy="0 0 ${pi*1}"/>
+      <geometry>
+        <mesh filename="package://open_manipulator_description/meshes/tartos_kamera3.dae" scale="1 1 1"/>
       </geometry>
     </collision>
